Commit message: Got maze imported into pushing env

File: assets/objects/maze/robot.urdf (robot description, URDF)
Before this commit: robot onshape, 1 links, 0 joints
Links:
- link part_1: mass 230.29999999999975557 -> 230.2999999999995282

Commit message: Maze and starting position are in a good spot

File: assets/objects/maze/robot.urdf (robot description, URDF)
Before this commit: robot onshape, 1 links, 0 joints
Links:
- link part_1: mass 230.2999999999995282 -> 151.69761309256711002

Commit message: Obstacles are ready

File: assets/objects/maze/robot.urdf (robot description, URDF)
Before this commit: robot onshape, 1 links, 0 joints
Links:
- link part_1: mass 230.2999999999995282 -> 261.02919742400149516

File: assets/objects/obstacle/obstacle.urdf (robot description, URDF)
Before this commit: robot obstacle.urdf, 1 links, 0 joints
Links:
- link baseLink: geometry collision box size=.05 .08 .1; visual box size=.05 0.08 .1
