Commit message: Working on making obstacle more reasonable fo pushing env:

File: assets/objects/cube/cube.urdf (robot description, URDF)
Before this commit: robot cube.urdf, 1 links, 0 joints
Links:
- link baseLink: geometry collision box size=.1 .1 .08; visual box size=.1 .1 .08

File: assets/objects/obstacle/obstacle.urdf (robot description, URDF)
Before this commit: robot obstacle.urdf, 1 links, 0 joints
Links:
- link baseLink: geometry collision box size=.05 .1 .1; visual box size=.05 0.1 .1
